File: kicad/irrigation-control-pcb/irrigation-control-pcb.kicad_pcb (KiCad board)
At the start: 2 copper layers, 49 x 26 mm, 7 parts

Commit message: pcbway print version 1.0
Parts:
- removed REF**: TerminalBlock_Phoenix_MKDS-1,5-4-5.08_1x04_P5.08mm_Horizont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, TerminalBlock_Phoenix:TerminalBlock_Phoenix_MKDS-1,5-4-5.08_1x04_P5.08mm_Horizontal
- removed REF**: TerminalBlock_Phoenix_MKDS-1,5-3-5.08_1x03_P5.08mm_Horizont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, TerminalBlock_Phoenix:TerminalBlock_Phoenix_MKDS-1,5-3-5.08_1x03_P5.08mm_Horizontal
- removed REF**: ESP_Test, kicad-custom-library:ESP_Test
- added 12V: x, TerminalBlock_Phoenix:TerminalBlock_Phoenix_MKDS-1,5-2-5.08_1x02_P5.08mm_Horizontal, F.Cu at (116.0, 80.0)
- added 3V3: TerminalBlock_Xinya_XY308-2.54-2P_1x02_P2.54mm_Horizontal, TerminalBlock:TerminalBlock_Xinya_XY308-2.54-2P_1x02_P2.54mm_Horizontal, F.Cu at (114.5, 99.5)
- added CTRL1: TerminalBlock_Xinya_XY308-2.54-3P_1x03_P2.54mm_Horizontal, TerminalBlock:TerminalBlock_Xinya_XY308-2.54-3P_1x03_P2.54mm_Horizontal, F.Cu at (103.9, 110.8)
- added ESPRESSIF: ESP_Test, kicad-custom-library:ESP_Test, F.Cu at (82.5, 89.5)
- added P1: x, TerminalBlock_Phoenix:TerminalBlock_Phoenix_MKDS-1,5-2-5.08_1x02_P5.08mm_Horizontal, F.Cu at (91.1, 67.3)
- added P2: x, TerminalBlock_Phoenix:TerminalBlock_Phoenix_MKDS-1,5-2-5.08_1x02_P5.08mm_Horizontal, F.Cu at (116.1, 67.3)
- added R1: Phoenix?, TerminalBlock_Phoenix:TerminalBlock_Phoenix_MKDS-1,5-2-5.08_1x02_P5.08mm_Horizontal, F.Cu at (78.5, 67.3)
- added R2: Phoenix?, TerminalBlock_Phoenix:TerminalBlock_Phoenix_MKDS-1,5-2-5.08_1x02_P5.08mm_Horizontal, F.Cu at (103.6, 67.3)
- added S2A: TerminalBlock_Xinya_XY308-2.54-4P_1x04_P2.54mm_Horizontal, TerminalBlock:TerminalBlock_Xinya_XY308-2.54-4P_1x04_P2.54mm_Horizontal, F.Cu at (81.9, 110.8)
- added S2B: TerminalBlock_Xinya_XY308-2.54-2P_1x02_P2.54mm_Horizontal, TerminalBlock:TerminalBlock_Xinya_XY308-2.54-2P_1x02_P2.54mm_Horizontal, F.Cu at (95.5, 110.8)
- added hole1: MountingHole_2.2mm_M2, MountingHole:MountingHole_2.2mm_M2, F.Cu at (60.5, 58.5)
- added hole1: MountingHole_2.2mm_M2, MountingHole:MountingHole_2.2mm_M2, F.Cu at (120.5, 58.5)
- added hole1: MountingHole_2.2mm_M2, MountingHole:MountingHole_2.2mm_M2, F.Cu at (120.5, 118.5)
- added hole1: MountingHole_2.2mm_M2, MountingHole:MountingHole_2.2mm_M2, F.Cu at (60.0, 118.5)
- PWR: renamed from REF**; value TerminalBlock_Phoenix_MKDS-1,5-2-5.08_1x02_P5.08mm_Horizontal -> x
- moved S1B 95.4 mm to (73.5, 110.8)
- moved S1A 74.2 mm to (60.9, 110.8)
- moved CTRL2 72.4 mm to (113.9, 110.8)
- moved PWR 42.0 mm to (66.0, 67.3), turned to 180 degrees
- renumbered REF** to CTRL2, REF** to S1A, REF** to S1B
Routing:
- net (no net): track 0.00 -> 506.9 mm
Other:
- board size 49 x 26 mm -> 67 x 67 mm
- board text removed: "VIN"
